File: main/main.sch (KiCad schematic (older format))
At the start: 16 parts

Commit message: picked_footprints
Parts:
- C1, C2, C3, C4: renamed from C?; footprint (none) -> Capacitor_SMD:C_1206_3216Metric_Pad1.42x1.75mm_HandSolder
- IN+1: renamed from IN+; footprint (none) -> Connector_PinHeader_2.54mm:PinHeader_1x01_P2.54mm_Vertical
- IN-1: renamed from IN-; footprint (none) -> Connector_PinHeader_2.54mm:PinHeader_1x01_P2.54mm_Vertical
- L1: renamed from L?; footprint (none) -> B82442T1103K050:B82442T1103K050
- LX1: renamed from LX; footprint (none) -> Connector_PinHeader_2.54mm:PinHeader_1x01_P2.54mm_Vertical
- MPPTSET1: renamed from MPPTSET; footprint (none) -> Connector_PinHeader_2.54mm:PinHeader_1x01_P2.54mm_Vertical
- OUT+1: renamed from OUT+; footprint (none) -> Connector_PinHeader_2.54mm:PinHeader_1x01_P2.54mm_Vertical
- OUT-1: renamed from OUT-; footprint (none) -> Connector_PinHeader_2.54mm:PinHeader_1x01_P2.54mm_Vertical
- R1, R2, R3: renamed from R?; footprint (none) -> Resistor_SMD:R_1206_3216Metric_Pad1.42x1.75mm_HandSolder
- U1: renamed from U?; footprint (none) -> Package_SO:TSSOP-8_4.4x3mm_P0.65mm; symbol CustomSymbols:SPV1040 -> main-rescue:SPV1040-CustomSymbols
- VCTRL1: renamed from VCTRL; footprint (none) -> Connector_PinHeader_2.54mm:PinHeader_1x01_P2.54mm_Vertical
Changed lines of the file:
@@
 EESchema Schematic File Version 4
+LIBS:main-cache
 EELAYER 29 0
 EELAYER END
@@
 $EndDescr
 $Comp
-L CustomSymbols:SPV1040 U?
+L main-rescue:SPV1040-CustomSymbols U1
 U 1 1 5DEFFC94
 P 5850 3700
-F 0 "U?" H 5800 4365 50  0000 C CNN
+F 0 "U1" H 5800 4365 50  0000 C CNN
 F 1 "SPV1040" H 5800 4274 50  0000 C CNN
-F 2 "" H 5850 3150 50  0001 C CNN
+F 2 "Package_SO:TSSOP-8_4.4x3mm_P0.65mm" H 5850 3150 50  0001 C CNN
 F 3 "" H 5850 3150 50  0001 C CNN
 	1    5850 3700
@@
 	5250 3900 5100 3900
 $Comp
-L power:GNDD #PWR?
+L power:GNDD #PWR03
 U 1 1 5DF00147
 P 5100 4450
-F 0 "#PWR?" H 5100 4200 50  0001 C CNN
+F 0 "#PWR03" H 5100 4200 50  0001 C CNN
 F 1 "GNDD" H 5104 4295 50  0000 C CNN
 F 2 "" H 5100 4450 50  0001 C CNN
@@
 $EndComp
 $Comp
-L Device:L L?
+L Device:L L1
 U 1 1 5DF0024B
 P 4650 3300
-F 0 "L?" V 4850 3300 50  0000 C CNN
+F 0 "L1" V 4850 3300 50  0000 C CNN
 F 1 "10u" V 4750 3300 50  0000 C CNN
-F 2 "" H 4650 3300 50  0001 C CNN
+F 2 "B82442T1103K050:B82442T1103K050" H 4650 3300 50  0001 C CNN
 F 3 "~" H 4650 3300 50  0001 C CNN
 	1    4650 3300
@@
 $EndComp
 $Comp
-L Device:R R?
+L Device:R R1
 U 1 1 5DF00C3E
 P 4350 3700
-F 0 "R?" V 4143 3700 50  0000 C CNN
+F 0 "R1" V 4143 3700 50  0000 C CNN
 F 1 "1K" V 4234 3700 50  0000 C CNN
-F 2 "" V 4280 3700 50  0001 C CNN
+F 2 "Resistor_SMD:R_1206_3216Metric_Pad1.42x1.75mm_HandSolder" V 4280 3700 50  0001 C CNN
 F 3 "~" H 4350 3700 50  0001 C CNN
 	1    4350 3700
@@
 $EndComp
 $Comp
-L Device:C C?
+L Device:C C1
 U 1 1 5DF03C7B
 P 3750 3950
-F 0 "C?" H 3865 3996 50  0000 L CNN
+F 0 "C1" H 3865 3996 50  0000 L CNN
 F 1 "100u" H 3865 3905 50  0000 L CNN
-F 2 "" H 3788 3800 50  0001 C CNN
+F 2 "Capacitor_SMD:C_1206_3216Metric_Pad1.42x1.75mm_HandSolder" H 3788 3800 50  0001 C CNN
 F 3 "~" H 3750 3950 50  0001 C CNN
 	1    3750 3950
@@
 $EndComp
 $Comp
-L power:GNDD #PWR?
+L power:GNDD #PWR01
 U 1 1 5DF0431D
 P 3750 4450
-F 0 "#PWR?" H 3750 4200 50  0001 C CNN
+F 0 "#PWR01" H 3750 4200 50  0001 C CNN
 F 1 "GNDD" H 3754 4295 50  0000 C CNN
 F 2 "" H 3750 4450 50  0001 C CNN
@@
 	6550 3500 6550 3300
 $Comp
-L Device:R R?
+L Device:R R2
 U 1 1 5DF04D7F
 P 7000 3600
-F 0 "R?" H 6930 3554 50  0000 R CNN
+F 0 "R2" H 6930 3554 50  0000 R CNN
 F 1 "768k" H 6930 3645 50  0000 R CNN
-F 2 "" V 6930 3600 50  0001 C CNN
+F 2 "Resistor_SMD:R_1206_3216Metric_Pad1.42x1.75mm_HandSolder" V 6930 3600 50  0001 C CNN
 F 3 "~" H 7000 3600 50  0001 C CNN
 	1    7000 3600
@@
 $EndComp
 $Comp
-L Device:R R?
+L Device:R R3
 U 1 1 5DF056B9
 P 7000 4150
-F 0 "R?" H 6930 4104 50  0000 R CNN
+F 0 "R3" H 6930 4104 50  0000 R CNN
 F 1 "330k" H 6930 4195 50  0000 R CNN
-F 2 "" V 6930 4150 50  0001 C CNN
+F 2 "Resistor_SMD:R_1206_3216Metric_Pad1.42x1.75mm_HandSolder" V 6930 4150 50  0001 C CNN
 F 3 "~" H 7000 4150 50  0001 C CNN
 	1    7000 4150
@@
 $EndComp
 $Comp
-L power:GNDD #PWR?
+L power:GNDD #PWR05
 U 1 1 5DF05A1C
 P 7000 4450
-F 0 "#PWR?" H 7000 4200 50  0001 C CNN
+F 0 "#PWR05" H 7000 4200 50  0001 C CNN
 F 1 "GNDD" H 7004 4295 50  0000 C CNN
 F 2 "" H 7000 4450 50  0001 C CNN
@@
 	7000 3900 7000 3750
 $Comp
-L Device:C C?
+L Device:C C3
 U 1 1 5DF067C0
 P 6500 4150
-F 0 "C?" H 6615 4196 50  0000 L CNN
+F 0 "C3" H 6615 4196 50  0000 L CNN
 F 1 "1n" H 6615 4105 50  0000 L CNN
-F 2 "" H 6538 4000 50  0001 C CNN
+F 2 "Capacitor_SMD:C_1206_3216Metric_Pad1.42x1.75mm_HandSolder" H 6538 4000 50  0001 C CNN
 F 3 "~" H 6500 4150 50  0001 C CNN
 	1    6500 4150
@@
 Connection ~ 6500 3900
 $Comp
-L power:GNDD #PWR?
+L power:GNDD #PWR04
 U 1 1 5DF06F65
 P 6500 4450
-F 0 "#PWR?" H 6500 4200 50  0001 C CNN
+F 0 "#PWR04" H 6500 4200 50  0001 C CNN
 F 1 "GNDD" H 6504 4295 50  0000 C CNN
 F 2 "" H 6500 4450 50  0001 C CNN
@@
 	3750 4450 3750 4100
 $Comp
-L Connector:TestPoint IN+
+L Connector:TestPoint IN+1
 U 1 1 5DF0C221
 P 3750 3300
-F 0 "IN+" V 3850 3700 50  0000 C CNN
+F 0 "IN+1" V 3850 3700 50  0000 C CNN
 F 1 "TestPoint" V 3750 3700 50  0000 C CNN
-F 2 "" H 3950 3300 50  0001 C CNN
+F 2 "Connector_PinHeader_2.54mm:PinHeader_1x01_P2.54mm_Vertical" H 3950 3300 50  0001 C CNN
 F 3 "~" H 3950 3300 50  0001 C CNN
 	1    3750 3300
@@
 $EndComp
 $Comp
-L Connector:TestPoint IN-
+L Connector:TestPoint IN-1
 U 1 1 5DF0CB9C
 P 3750 4450
-F 0 "IN-" V 3850 4800 50  0000 C CNN
+F 0 "IN-1" V 3850 4800 50  0000 C CNN
 F 1 "TestPoint" V 3750 4800 50  0000 C CNN
-F 2 "" H 3950 4450 50  0001 C CNN
+F 2 "Connector_PinHeader_2.54mm:PinHeader_1x01_P2.54mm_Vertical" H 3950 4450 50  0001 C CNN
 F 3 "~" H 3950 4450 50  0001 C CNN
 	1    3750 4450
@@
 Connection ~ 3750 4450
 $Comp
-L Device:C C?
+L Device:C C4
 U 1 1 5DF0D320
 P 7900 3900
-F 0 "C?" H 8015 3946 50  0000 L CNN
+F 0 "C4" H 8015 3946 50  0000 L CNN
 F 1 "100u" H 8015 3855 50  0000 L CNN
-F 2 "" H 7938 3750 50  0001 C CNN
+F 2 "Capacitor_SMD:C_1206_3216Metric_Pad1.42x1.75mm_HandSolder" H 7938 3750 50  0001 C CNN
 F 3 "~" H 7900 3900 50  0001 C CNN
 	1    7900 3900
@@
 	7900 3750 7900 3300
 $Comp
-L power:GNDD #PWR?
+L power:GNDD #PWR06
 U 1 1 5DF0DCB1
 P 7900 4450
-F 0 "#PWR?" H 7900 4200 50  0001 C CNN
+F 0 "#PWR06" H 7900 4200 50  0001 C CNN
 F 1 "GNDD" H 7904 4295 50  0000 C CNN
 F 2 "" H 7900 4450 50  0001 C CNN
@@
 	7900 4450 7900 4050
 $Comp
-L Connector:TestPoint OUT+
+L Connector:TestPoint OUT+1
 U 1 1 5DF0E3DD
 P 7900 3300
-F 0 "OUT+" V 8000 3700 50  0000 C CNN
+F 0 "OUT+1" V 8000 3700 50  0000 C CNN
 F 1 "TestPoint" V 7900 3700 50  0000 C CNN
-F 2 "" H 8100 3300 50  0001 C CNN
+F 2 "Connector_PinHeader_2.54mm:PinHeader_1x01_P2.54mm_Vertical" H 8100 3300 50  0001 C CNN
 F 3 "~" H 8100 3300 50  0001 C CNN
 	1    7900 3300
@@
 Connection ~ 7900 3300
 $Comp
-L Connector:TestPoint OUT-
+L Connector:TestPoint OUT-1
 U 1 1 5DF0EE0A
 P 7900 4450
-F 0 "OUT-" V 8000 4800 50  0000 C CNN
+F 0 "OUT-1" V 8000 4800 50  0000 C CNN
 F 1 "TestPoint" V 7900 4800 50  0000 C CNN
-F 2 "" H 8100 4450 50  0001 C CNN
+F 2 "Connector_PinHeader_2.54mm:PinHeader_1x01_P2.54mm_Vertical" H 8100 4450 50  0001 C CNN
 F 3 "~" H 8100 4450 50  0001 C CNN
 	1    7900 4450
@@
 	5100 3700 5250 3700
 $Comp
-L Device:C C?
+L Device:C C2
 U 1 1 5DF18322
 P 4700 4150
-F 0 "C?" H 4815 4196 50  0000 L CNN
+F 0 "C2" H 4815 4196 50  0000 L CNN
 F 1 "1n" H 4815 4105 50  0000 L CNN
-F 2 "" H 4738 4000 50  0001 C CNN
+F 2 "Capacitor_SMD:C_1206_3216Metric_Pad1.42x1.75mm_HandSolder" H 4738 4000 50  0001 C CNN
 F 3 "~" H 4700 4150 50  0001 C CNN
 	1    4700 4150
@@
 $EndComp
 $Comp
-L power:GNDD #PWR?
+L power:GNDD #PWR02
 U 1 1 5DF1832D
 P 4700 4450
-F 0 "#PWR?" H 4700 4200 50  0001 C CNN
+F 0 "#PWR02" H 4700 4200 50  0001 C CNN
 F 1 "GNDD" H 4704 4295 50  0000 C CNN
 F 2 "" H 4700 4450 50  0001 C CNN
@@
 	6500 3900 7000 3900
 $Comp
-L Connector:TestPoint VCTRL
+L Connector:TestPoint VCTRL1
 U 1 1 5DF20AB3
 P 7000 3900
-F 0 "VCTRL" V 7100 4300 50  0000 C CNN
+F 0 "VCTRL1" V 7100 4300 50  0000 C CNN
 F 1 "TestPoint" V 7000 4300 50  0000 C CNN
-F 2 "" H 7200 3900 50  0001 C CNN
+F 2 "Connector_PinHeader_2.54mm:PinHeader_1x01_P2.54mm_Vertical" H 7200 3900 50  0001 C CNN
 F 3 "~" H 7200 3900 50  0001 C CNN
 	1    7000 3900
@@
 $EndComp
 $Comp
-L Connector:TestPoint MPPTSET
+L Connector:TestPoint MPPTSET1
 U 1 1 5DF20F1E
 P 4900 3700
-F 0 "MPPTSET" H 4900 4000 50  0000 C CNN
+F 0 "MPPTSET1" H 4900 4000 50  0000 C CNN
 F 1 "TestPoint" H 4900 3900 50  0000 C CNN
-F 2 "" H 5100 3700 50  0001 C CNN
+F 2 "Connector_PinHeader_2.54mm:PinHeader_1x01_P2.54mm_Vertical" H 5100 3700 50  0001 C CNN
 F 3 "~" H 5100 3700 50  0001 C CNN
 	1    4900 3700
@@
 	4900 3700 5100 3700
 $Comp
-L Connector:TestPoint LX
+L Connector:TestPoint LX1
 U 1 1 5DF21880
 P 5200 3300
-F 0 "LX" H 5200 3550 50  0000 C CNN
+F 0 "LX1" H 5200 3550 50  0000 C CNN
 F 1 "TestPoint" H 5200 3650 50  0000 C CNN
-F 2 "" H 5400 3300 50  0001 C CNN
+F 2 "Connector_PinHeader_2.54mm:PinHeader_1x01_P2.54mm_Vertical" H 5400 3300 50  0001 C CNN
 F 3 "~" H 5400 3300 50  0001 C CNN
 	1    5200 3300
