File: main/main.kicad_pcb (KiCad board)
At the start: 2 copper layers, 16 parts, among them U1 SPV1040

Commit message: progress
Parts:
- removed LX1, OUT-1: TestPoint, Connector_PinHeader_2.54mm:PinHeader_1x01_P2.54mm_Vertical
- moved L1 70.7 mm to (88.0, 123.2)
- moved R3 68.9 mm to (106.9, 122.2), turned to 90 degrees
- moved C3 65.0 mm to (101.8, 120.6), turned to 270 degrees
- moved IN-1 64.7 mm to (91.4, 127.9)
- moved C1 64.5 mm to (91.4, 117.2), turned to 270 degrees
- moved U1 62.0 mm to (98.8, 115.9)
- moved R2 61.4 mm to (106.9, 117.1), turned to 90 degrees
- moved C4 60.5 mm to (104.1, 117.2), turned to 270 degrees
- moved R1 59.5 mm to (89.6, 113.3), turned to 180 degrees
- moved IN+1 59.1 mm to (84.0, 113.7)
- moved OUT+1 57.9 mm to (110.9, 115.6)
- moved MPPTSET1 57.3 mm to (98.5, 111.9)
- moved VCTRL1 55.8 mm to (98.3, 119.1)
- moved C2 53.1 mm to (93.3, 111.9), turned to 90 degrees
Routing:
- net Net-(C4-Pad1): track 0.00 -> 18.2 mm
- net Net-(C2-Pad1): track 0.00 -> 16.2 mm
- net Net-(C1-Pad1): track 0.00 -> 15.0 mm
- net Net-(C3-Pad1): track 0.00 -> 14.4 mm
- net GNDD: track 0.00 -> 9.19 mm
- net Net-(L1-Pad2): track 0.00 -> 8.47 mm
Other:
- net class 0.75 added: clearance 0.2, trace_width 0.75, via_dia 0.8, via_drill 0.4

Commit message: gerber
Parts:
- added LX1: TestPoint, Connector_PinHeader_2.54mm:PinHeader_1x01_P2.54mm_Vertical, F.Cu at (129.5, 77.5)
- added OUT-1: TestPoint, Connector_PinHeader_2.54mm:PinHeader_1x01_P2.54mm_Vertical, F.Cu at (140.9, 86.5)
- moved VCTRL1 74.3 mm to (157.8, 74.6)
- moved L1 69.2 mm to (134.5, 71.9), turned to 270 degrees
- moved MPPTSET1 65.7 mm to (152.6, 74.6)
- moved R1 64.6 mm to (135.9, 68.4)
- moved R3 64.4 mm to (155.4, 79.9)
- moved C3 64.4 mm to (151.7, 79.9)
- moved R2 64.3 mm to (159.3, 79.9), turned to 270 degrees
- moved C2 63.4 mm to (142.0, 71.3)
- moved IN-1 63.2 mm to (135.1, 82.2)
- moved C1 62.9 mm to (139.5, 76.6)
- moved IN+1 61.9 mm to (129.6, 71.9)
- moved U1 61.3 mm to (146.2, 77.0)
- moved C4 50.9 mm to (140.9, 81.9)
- moved OUT+1 47.3 mm to (145.3, 83.2)
Routing:
- net GNDD: track 9.19 -> 31.3 mm, vias 0 -> 10
- net Net-(C4-Pad1): track 18.2 -> 32.5 mm, vias 0 -> 2
- net Net-(C2-Pad1): track 16.2 -> 25.8 mm, vias 0 -> 1
- net Net-(L1-Pad2): track 8.47 -> 14.4 mm
- added copper zone on B.Cu, net GNDD
- added copper zone on F.Cu, net GNDD
Other:
- board outline added: 79 x 67 mm
